File: laprobe/laprobe.kicad_pcb (KiCad board)
At the start: 2 copper layers, 90 x 60 mm, 281 parts, among them J101 Conn_02x04_Row_Letter_Last, J102 Conn_02x04_Row_Letter_Last, J103 Conn_02x04_Row_Letter_Last, J104 Conn_02x04_Row_Letter_Last, J105 Conn_02x25_Odd_Even, U201 LMH7324, U301 LMH7324, U401 LMH7324, U501 LMH7324

Commit message: Checkpoint: All but frozen ch0
Parts:
- C213, C214, C215, C216, C217, C218, C219, C220, C221, C222, C223, C224: moved to B.Cu
- moved C209 94.1 mm to (101.7, 46.8)
- moved C224 93.3 mm to (94.7, 46.3), turned to -90 degrees
- moved C210 93.1 mm to (101.7, 50.5)
- moved C235 91.5 mm to (94.7, 43.2), turned to 90 degrees
- moved C221 89.2 mm to (97.8, 46.3), turned to -90 degrees
- moved C222 87.5 mm to (97.8, 51.0), turned to 90 degrees
- moved C223 87.5 mm to (94.7, 51.0), turned to 90 degrees
- moved C236 87.0 mm to (90.8, 48.6), turned to 180 degrees
- moved C234 85.2 mm to (91.4, 46.1), turned to 90 degrees
- moved C220 83.0 mm to (93.9, 48.6), turned to 180 degrees
- moved C218 82.3 mm to (98.6, 48.6)
- moved C230 81.7 mm to (101.7, 48.6)
- moved C219 80.9 mm to (96.2, 51.0), turned to -90 degrees
- moved C217 80.6 mm to (96.2, 46.3), turned to 90 degrees
- moved C233 79.6 mm to (96.2, 54.1), turned to -90 degrees
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Connections:
- C202 pad 2: Net-(U201B-+) -> Net-(U201D-+)
- C204 pad 2: Net-(U201D-+) -> Net-(U201B-+)
- C206 pad 1: Net-(U201B-+) -> Net-(U201D-+)
- C208 pad 1: Net-(U201D-+) -> Net-(U201B-+)
- C302 pad 2: Net-(U301B-+) -> Net-(U301D-+)
- C304 pad 2: Net-(U301D-+) -> Net-(U301B-+)
- C306 pad 1: Net-(U301B-+) -> Net-(U301D-+)
- C308 pad 1: Net-(U301D-+) -> Net-(U301B-+)
- C402 pad 2: Net-(U401B-+) -> Net-(U401D-+)
- C404 pad 2: Net-(U401D-+) -> Net-(U401B-+)
- C406 pad 1: Net-(U401B-+) -> Net-(U401D-+)
- C408 pad 1: Net-(U401D-+) -> Net-(U401B-+)
- C502 pad 2: Net-(U501B-+) -> Net-(U501D-+)
- C504 pad 2: Net-(U501D-+) -> Net-(U501B-+)
- C506 pad 1: Net-(U501B-+) -> Net-(U501D-+)
- C508 pad 1: Net-(U501D-+) -> Net-(U501B-+)
- R210 pad 2: Net-(U201B-+) -> Net-(U201D-+)
- R212 pad 2: Net-(U201D-+) -> Net-(U201B-+)
- R214 pad 1: Net-(U201B-+) -> Net-(U201D-+)
- R216 pad 1: Net-(U201D-+) -> Net-(U201B-+)
- R218 pad 1: Net-(U201B-Q) -> Net-(U201D-Q)
- R220 pad 1: Net-(U201D-Q) -> Net-(U201B-Q)
- R222 pad 1: Net-(U201B-~{Q}) -> Net-(U201D-~{Q})
- R224 pad 1: Net-(U201D-~{Q}) -> Net-(U201B-~{Q})
- R227 pad 1: Net-(U201B-Q) -> Net-(U201D-Q)
- R228 pad 1: Net-(U201B-~{Q}) -> Net-(U201D-~{Q})
- R231 pad 1: Net-(U201D-Q) -> Net-(U201B-Q)
- R232 pad 1: Net-(U201D-~{Q}) -> Net-(U201B-~{Q})
- R310 pad 2: Net-(U301B-+) -> Net-(U301D-+)
- R312 pad 2: Net-(U301D-+) -> Net-(U301B-+)
- R314 pad 1: Net-(U301B-+) -> Net-(U301D-+)
- R316 pad 1: Net-(U301D-+) -> Net-(U301B-+)
- R318 pad 1: Net-(U301B-Q) -> Net-(U301D-Q)
- R320 pad 1: Net-(U301D-Q) -> Net-(U301B-Q)
- R322 pad 1: Net-(U301B-~{Q}) -> Net-(U301D-~{Q})
- R324 pad 1: Net-(U301D-~{Q}) -> Net-(U301B-~{Q})
- R327 pad 1: Net-(U301B-Q) -> Net-(U301D-Q)
- R328 pad 1: Net-(U301B-~{Q}) -> Net-(U301D-~{Q})
- R331 pad 1: Net-(U301D-Q) -> Net-(U301B-Q)
- R332 pad 1: Net-(U301D-~{Q}) -> Net-(U301B-~{Q})
- R410 pad 2: Net-(U401B-+) -> Net-(U401D-+)
- R412 pad 2: Net-(U401D-+) -> Net-(U401B-+)
- R414 pad 1: Net-(U401B-+) -> Net-(U401D-+)
- R416 pad 1: Net-(U401D-+) -> Net-(U401B-+)
- R418 pad 1: Net-(U401B-Q) -> Net-(U401D-Q)
- R420 pad 1: Net-(U401D-Q) -> Net-(U401B-Q)
- R422 pad 1: Net-(U401B-~{Q}) -> Net-(U401D-~{Q})
- R424 pad 1: Net-(U401D-~{Q}) -> Net-(U401B-~{Q})
- R427 pad 1: Net-(U401B-Q) -> Net-(U401D-Q)
- R428 pad 1: Net-(U401B-~{Q}) -> Net-(U401D-~{Q})
- R431 pad 1: Net-(U401D-Q) -> Net-(U401B-Q)
- R432 pad 1: Net-(U401D-~{Q}) -> Net-(U401B-~{Q})
- R510 pad 2: Net-(U501B-+) -> Net-(U501D-+)
- R512 pad 2: Net-(U501D-+) -> Net-(U501B-+)
- R514 pad 1: Net-(U501B-+) -> Net-(U501D-+)
- R516 pad 1: Net-(U501D-+) -> Net-(U501B-+)
- R518 pad 1: Net-(U501B-Q) -> Net-(U501D-Q)
- R520 pad 1: Net-(U501D-Q) -> Net-(U501B-Q)
- R522 pad 1: Net-(U501B-~{Q}) -> Net-(U501D-~{Q})
- R524 pad 1: Net-(U501D-~{Q}) -> Net-(U501B-~{Q})
- R527 pad 1: Net-(U501B-Q) -> Net-(U501D-Q)
- R528 pad 1: Net-(U501B-~{Q}) -> Net-(U501D-~{Q})
- R531 pad 1: Net-(U501D-Q) -> Net-(U501B-Q)
- R532 pad 1: Net-(U501D-~{Q}) -> Net-(U501B-~{Q})
